File: Hardware/Proto Kicad/mod-player.kicad_sch (KiCad schematic)
At the start: 95 parts, among them J1 USB_C_Receptacle_USB2.0, J2 Micro_SD_Card_Det1, J3 Conn_01x03_MountingPin, J4 Conn_01x01_Pin, J5 Conn_01x01_Pin, Q1 NMOS, Q2 AO3401A, Q3 NMOS, Q4 NMOS, Q5 NMOS, Q6 NMOS, Q7 NMOS, Q8 NMOS, SW2 SW_MEC_5E, SW3 SW_MEC_5E, SW4 SW_MEC_5E, SW5 SW_MEC_5E, SW6 SW_MEC_5E, SW7 SW_Push_DPDT, U1 RP2040, U2 MT3608, U3 AMS1117-3.3, U4 W25Q32JVSS, U5 MAX98357AETE_T, Y1 12MHZ

Commit message: more hardware
Parts:
- removed R15, R16, R17: 1k, Resistor_SMD:R_0603_1608Metric, symbol Device:R
- removed R4: R, Resistor_SMD:R_0603_1608Metric, symbol Device:R
- added J7: Conn_02x06_Odd_Even, Connector_PinHeader_2.54mm:PinHeader_2x06_P2.54mm_Vertical_SMD, symbol Connector_Generic:Conn_02x06_Odd_Even
- added RN2: R_Pack04_Split, Resistor_SMD:R_Array_Convex_4x0402, symbol Device:R_Pack04_Split
Connections:
- net +3V3: now also J7.11 (Pin_11), RN2.1 (R1.1), RN2.2 (R2.1), RN2.3 (R3.1)
- net GND: now also J7.12 (Pin_12)
- net SW1: now also RN2.6 (R3.2)
- net SW2: now also RN2.8 (R1.2)
- net SW3: now also RN2.7 (R2.2)
- net GP16: now reaches U1.27 (GPIO16)
- net GP16: now also J7.6 (Pin_6)
- net GP17: now reaches U1.28 (GPIO17)
- net GP17: now also J7.8 (Pin_8)
- net GP18: now reaches U1.29 (GPIO18)
- net GP18: now also J7.10 (Pin_10)
- net GP19: now reaches U1.30 (GPIO19)
- net GP19: now also J7.9 (Pin_9)
- net GP23: now reaches U1.35 (GPIO23)
- net GP23: now also J7.7 (Pin_7)
- net GP24: now reaches U1.36 (GPIO24)
- net GP24: now also J7.5 (Pin_5)
- net GP25: now reaches U1.37 (GPIO25)
- net GP25: now also J7.3 (Pin_3)
- net GP27: now reaches U1.39 (GPIO27_ADC1)
- net GP27: now also J7.1 (Pin_1)
- net GP28: now reaches U1.40 (GPIO28_ADC2)
- net GP28: now also J7.2 (Pin_2)
- net GP29: now reaches U1.41 (GPIO29_ADC3)
- net GP29: now also J7.4 (Pin_4)
