File: Hardware/mod-badge-inercia/mod-badge-inercia.kicad_sch (KiCad schematic)
At the start: 72 parts, among them J1 USB_C_Receptacle_USB2.0, J2 Micro_SD_Card_Det1, J3 Conn_01x03_MountingPin, J4 Conn_01x01_Pin, J5 Conn_01x01_Pin, J7 Conn_02x06_Odd_Even, Q2 AO3401A, SW2 SW_MEC_5E, SW3 SW_MEC_5E, SW4 SW_MEC_5E, SW5 SW_MEC_5E, SW6 SW_MEC_5E, SW7 SW_Push_DPDT, U1 RP2040, U2 MT3608, U3 AMS1117-3.3, U4 W25Q32JVSS, U5 MAX98357AETE_T, Y1 12MHZ

Commit message: boards exported and sent to fab
Parts:
- removed R53: 0, Resistor_SMD:R_0603_1608Metric, symbol Device:R
Connections:
- net +3V3: now also C18.2, C19.2, U5.7 (VDD), U5.8 (VDD)
